Commit message: Wheel alligned

File: description/robot_main.xacro (robot description, xacro)
@@ -23,5 +23,5 @@
             <origin xyz = "0.135 0 0.07"/>
             <geometry>
-                <box size = "0.27 0.168 0.14" />
+                <box size = "0.27 0.168 0.10577" />
             </geometry>
             <material name = "white"/>
@@ -32,5 +32,5 @@
         <parent link = "base_link"/>
         <child link = "r_wheel"/>
-        <origin xyz = "0.09647 -0.1025 0.01727" rpy = "${pi/2} 0 0"/>
+        <origin xyz = "0.135 -0.1025 0.01727" rpy = "${pi/2} 0 0"/>
         <axis xyz = "0 0 -1"/>
     </joint>
@@ -47,5 +47,5 @@
         <parent link = "base_link"/>
         <child link = "l_wheel"/>
-        <origin xyz = "0.09647 0.1025 0.01727" rpy = "-${pi/2} 0 0"/>
+        <origin xyz = "0.135 0.1025 0.01727" rpy = "-${pi/2} 0 0"/>
         <axis xyz = "0 0 1"/>
     </joint>

Commit message: castor cylinder added

File: description/robot_main.xacro (robot description, xacro)
@@ -32,5 +32,5 @@
         <parent link = "base_link"/>
         <child link = "r_wheel"/>
-        <origin xyz = "0.135 -0.1025 0.01727" rpy = "${pi/2} 0 0"/>
+        <origin xyz = "0.135 -0.1025 0.03454" rpy = "${pi/2} 0 0"/>
         <axis xyz = "0 0 -1"/>
     </joint>
@@ -47,5 +47,5 @@
         <parent link = "base_link"/>
         <child link = "l_wheel"/>
-        <origin xyz = "0.135 0.1025 0.01727" rpy = "-${pi/2} 0 0"/>
+        <origin xyz = "0.135 0.1025 0.03454" rpy = "-${pi/2} 0 0"/>
         <axis xyz = "0 0 1"/>
     </joint>
@@ -58,3 +58,31 @@
         </visual>
     </link>
+    <!-- left cylinder-->
+    <joint name = "l_cylinder_joint" type = "fixed">
+       <parent link = "body"/>
+       <child link = "l_cylinder"/>
+       <origin xyz = "0.045 0.059 0.010615" rpy = "0 0 0"/>
+    </joint>
+    <link name = "l_cylinder">
+         <visual>
+            <geometry>
+                <cylinder radius = "0.015" length = "0.02123"/>
+            </geometry>
+            <material name = "black"/>
+        </visual>
+    </link>
+     <!-- right cylinder-->
+    <joint name = "r_cylinder_joint" type = "fixed">
+       <parent link = "body"/>
+       <child link = "r_cylinder"/>
+       <origin xyz = "0.045 -0.059 0.010615" rpy = "0 0 0"/>
+    </joint>
+    <link name = "r_cylinder">
+         <visual>
+            <geometry>
+                <cylinder radius = "0.015" length = "0.02123"/>
+            </geometry>
+            <material name = "black"/>
+        </visual>
+    </link>
 </robot>

Commit message: inertia

File: description/robot_main.xacro (robot description, xacro)
@@ -1,4 +1,5 @@
 <?xml version="1.0"?>
 <robot xmlns:xacro="http://www.ros.org/wiki/xacro"  name="robot">
+    <xacro:include filename = "inertial_macros.xacro"/>
     <material name = "white">
         <color rgba = "1 1 1 1" />
@@ -27,4 +28,13 @@
             <material name = "white"/>
         </visual>
+        <collision>
+            <origin xyz = "0.135 0 0.07"/>
+            <geometry>
+                <box size = "0.27 0.168 0.10577" />
+            </geometry>
+        </collision>
+        <xacro:inertial_box mass="0.7" x="0.27" y="0.168" z="0.10577">
+            <origin xyz = "0.135 0 0.07" rpy = "0 0 0"/>
+        </xacro:inertial_box>
     </link>
     <!-- right wheel link -->
@@ -42,4 +52,12 @@
             <material name = "black"/>
         </visual>
+        <collision>
+            <geometry>
+                <cylinder radius = "0.04" length = "0.037"/>
+            </geometry>
+        </collision>
+        <xacro:inertial_cylinder mass="0.044" length="0.037" radius="0.04">
+            <origin xyz = "0 0 0" rpy = "0 0 0 "/>
+        </xacro:inertial_cylinder>
     </link>
     <!-- left wheel link -->
@@ -57,4 +75,12 @@
             <material name = "black"/>
         </visual>
+        <collision>
+            <geometry>
+                <cylinder radius = "0.04" length = "0.037"/>
+            </geometry>
+        </collision>
+        <xacro:inertial_cylinder mass="0.044" length="0.037" radius="0.04">
+            <origin xyz = "0 0 0" rpy = "0 0 0 "/>
+        </xacro:inertial_cylinder>
     </link>
     <!-- left cylinder-->
@@ -71,4 +97,12 @@
             <material name = "black"/>
         </visual>
+        <collision>
+            <geometry>
+                <cylinder radius = "0.015" length = "0.02123"/>
+            </geometry>
+        </collision>
+        <xacro:inertial_cylinder mass="0.02" radius="0.015" length="0.02123">
+            <origin xyz = "0 0 0" rpy = "0 0 0 "/>
+        </xacro:inertial_cylinder>
     </link>
      <!-- right cylinder-->
@@ -85,4 +119,57 @@
             <material name = "black"/>
         </visual>
+        <collision>
+            <geometry>
+                <cylinder radius = "0.015" length = "0.02123"/>
+            </geometry>
+            <material name = "black"/>
+        </collision>
+        <xacro:inertial_cylinder mass="0.02" radius="0.015" length="0.02123">
+            <origin xyz = "0 0 0" rpy = "0 0 0 "/>
+        </xacro:inertial_cylinder>
+    </link>
+    <!-- left castor-->
+    <joint name = "l_castor_joint" type = "fixed">
+        <parent link = "l_cylinder"/>
+        <child link = "l_castor"/>
+        <origin xyz = "0 0 -0.010615" rpy = "0 0 0"/>
+    </joint>
+    <link name = "l_castor">
+         <visual>
+            <geometry>
+                <sphere radius = "0.015" />
+            </geometry>
+            <material name = "orange"/>
+        </visual>
+        <collision>
+            <geometry>
+                <sphere radius = "0.015" />
+            </geometry>
+        </collision>
+        <xacro:inertial_sphere mass="0.03" radius="0.015">
+            <origin xyz = "0 0 0" rpy = "0 0 0 "/>
+        </xacro:inertial_sphere>
+    </link>
+    <!-- right castor-->
+    <joint name = "r_castor_joint" type = "fixed">
+        <parent link = "r_cylinder"/>
+        <child link = "r_castor"/>
+        <origin xyz = "0 0 -0.010615" rpy = "0 0 0"/>
+    </joint>
+    <link name = "r_castor">
+         <visual>
+            <geometry>
+                <sphere radius = "0.015" />
+            </geometry>
+            <material name = "orange"/>
+        </visual>
+        <collision>
+            <geometry>
+                <sphere radius = "0.015" />
+            </geometry>
+        </collision>
+        <xacro:inertial_sphere mass="0.03" radius="0.015">
+            <origin xyz = "0 0 0" rpy = "0 0 0 "/>
+        </xacro:inertial_sphere>
     </link>
 </robot>

Commit message: gazebo launch

File: description/robot_main.xacro (robot description, xacro)
@@ -42,5 +42,5 @@
         <parent link = "base_link"/>
         <child link = "r_wheel"/>
-        <origin xyz = "0.135 -0.1025 0.03454" rpy = "${pi/2} 0 0"/>
+        <origin xyz = "0.135 -0.094 0.03454" rpy = "${pi/2} 0 0"/>
         <axis xyz = "0 0 -1"/>
     </joint>
@@ -48,5 +48,5 @@
         <visual>
             <geometry>
-                <cylinder radius = "0.04" length = "0.037"/>
+                <cylinder radius = "0.035" length = "0.020"/>
             </geometry>
             <material name = "black"/>
@@ -54,8 +54,8 @@
         <collision>
             <geometry>
-                <cylinder radius = "0.04" length = "0.037"/>
+                <cylinder radius = "0.035" length = "0.020"/>
             </geometry>
         </collision>
-        <xacro:inertial_cylinder mass="0.044" length="0.037" radius="0.04">
+        <xacro:inertial_cylinder mass="0.04" length="0.02" radius="0.035">
             <origin xyz = "0 0 0" rpy = "0 0 0 "/>
         </xacro:inertial_cylinder>
@@ -65,5 +65,5 @@
         <parent link = "base_link"/>
         <child link = "l_wheel"/>
-        <origin xyz = "0.135 0.1025 0.03454" rpy = "-${pi/2} 0 0"/>
+        <origin xyz = "0.135 0.094 0.03454" rpy = "-${pi/2} 0 0"/>
         <axis xyz = "0 0 1"/>
     </joint>
@@ -71,5 +71,5 @@
         <visual>
             <geometry>
-                <cylinder radius = "0.04" length = "0.037"/>
+                <cylinder radius = "0.035" length = "0.02"/>
             </geometry>
             <material name = "black"/>
@@ -77,21 +77,21 @@
         <collision>
             <geometry>
-                <cylinder radius = "0.04" length = "0.037"/>
+                <cylinder radius = "0.035" length = "0.02"/>
             </geometry>
         </collision>
-        <xacro:inertial_cylinder mass="0.044" length="0.037" radius="0.04">
+        <xacro:inertial_cylinder mass="0.04" length="0.02" radius="0.035">
             <origin xyz = "0 0 0" rpy = "0 0 0 "/>
         </xacro:inertial_cylinder>
     </link>
-    <!-- left cylinder-->
+    <!-- cylinder-->
     <joint name = "l_cylinder_joint" type = "fixed">
        <parent link = "body"/>
        <child link = "l_cylinder"/>
-       <origin xyz = "0.045 0.059 0.010615" rpy = "0 0 0"/>
+       <origin xyz = "0.045 0 0.010615" rpy = "0 0 0"/>
     </joint>
     <link name = "l_cylinder">
          <visual>
             <geometry>
-                <cylinder radius = "0.015" length = "0.02123"/>
+                <cylinder radius = "0.0075" length = "0.01023"/>
             </geometry>
             <material name = "black"/>
@@ -99,44 +99,21 @@
         <collision>
             <geometry>
-                <cylinder radius = "0.015" length = "0.02123"/>
+                <cylinder radius = "0.0075" length = "0.01023"/>
             </geometry>
         </collision>
-        <xacro:inertial_cylinder mass="0.02" radius="0.015" length="0.02123">
+        <xacro:inertial_cylinder mass="0.001" radius="0.0075" length="0.01023">
             <origin xyz = "0 0 0" rpy = "0 0 0 "/>
         </xacro:inertial_cylinder>
     </link>
-     <!-- right cylinder-->
-    <joint name = "r_cylinder_joint" type = "fixed">
-       <parent link = "body"/>
-       <child link = "r_cylinder"/>
-       <origin xyz = "0.045 -0.059 0.010615" rpy = "0 0 0"/>
-    </joint>
-    <link name = "r_cylinder">
-         <visual>
-            <geometry>
-                <cylinder radius = "0.015" length = "0.02123"/>
-            </geometry>
-            <material name = "black"/>
-        </visual>
-        <collision>
-            <geometry>
-                <cylinder radius = "0.015" length = "0.02123"/>
-            </geometry>
-            <material name = "black"/>
-        </collision>
-        <xacro:inertial_cylinder mass="0.02" radius="0.015" length="0.02123">
-            <origin xyz = "0 0 0" rpy = "0 0 0 "/>
-        </xacro:inertial_cylinder>
-    </link>
-    <!-- left castor-->
+    <!-- ball castor-->
     <joint name = "l_castor_joint" type = "fixed">
         <parent link = "l_cylinder"/>
         <child link = "l_castor"/>
-        <origin xyz = "0 0 -0.010615" rpy = "0 0 0"/>
+        <origin xyz = "0 0 -0.004" rpy = "0 0 0"/>
     </joint>
     <link name = "l_castor">
          <visual>
             <geometry>
-                <sphere radius = "0.015" />
+                <sphere radius = "0.0075" />
             </geometry>
             <material name = "orange"/>
@@ -144,30 +121,8 @@
         <collision>
             <geometry>
-                <sphere radius = "0.015" />
+                <sphere radius = "0.0075" />
             </geometry>
         </collision>
-        <xacro:inertial_sphere mass="0.03" radius="0.015">
-            <origin xyz = "0 0 0" rpy = "0 0 0 "/>
-        </xacro:inertial_sphere>
-    </link>
-    <!-- right castor-->
-    <joint name = "r_castor_joint" type = "fixed">
-        <parent link = "r_cylinder"/>
-        <child link = "r_castor"/>
-        <origin xyz = "0 0 -0.010615" rpy = "0 0 0"/>
-    </joint>
-    <link name = "r_castor">
-         <visual>
-            <geometry>
-                <sphere radius = "0.015" />
-            </geometry>
-            <material name = "orange"/>
-        </visual>
-        <collision>
-            <geometry>
-                <sphere radius = "0.015" />
-            </geometry>
-        </collision>
-        <xacro:inertial_sphere mass="0.03" radius="0.015">
+        <xacro:inertial_sphere mass="0.01" radius="0.0075">
             <origin xyz = "0 0 0" rpy = "0 0 0 "/>
         </xacro:inertial_sphere>
