Commit message: gazebo and rviz odom

File: description/robot.urdf.xacro (robot description, xacro)
@@ -2,3 +2,4 @@
 <robot xmlns:xacro="http://www.ros.org/wiki/xacro"  name="robot">
     <xacro:include filename = "robot_main.xacro"/>
+    <xacro:include filename="gazebo_control.xacro"/>
 </robot>

File: description/robot_main.xacro (robot description, xacro)
@@ -38,4 +38,7 @@
         </xacro:inertial_box>
     </link>
+    <gazebo reference="body">
+        <material>Gazebo/White</material>
+    </gazebo>
     <!-- right wheel link -->
     <joint name = "r_wheel_joint" type = "continuous">
@@ -61,4 +64,7 @@
         </xacro:inertial_cylinder>
     </link>
+    <gazebo reference="r_wheel">
+        <material>Gazebo/Black</material>
+    </gazebo>
     <!-- left wheel link -->
     <joint name = "l_wheel_joint" type = "continuous">
@@ -84,11 +90,14 @@
         </xacro:inertial_cylinder>
     </link>
+    <gazebo reference="l_wheel">
+        <material>Gazebo/Black</material>
+    </gazebo>
     <!-- cylinder-->
-    <joint name = "l_cylinder_joint" type = "fixed">
+    <joint name = "cylinder_joint" type = "fixed">
        <parent link = "body"/>
-       <child link = "l_cylinder"/>
+       <child link = "cylinder"/>
        <origin xyz = "0.045 0 0.010615" rpy = "0 0 0"/>
     </joint>
-    <link name = "l_cylinder">
+    <link name = "cylinder">
          <visual>
             <geometry>
@@ -106,11 +115,14 @@
         </xacro:inertial_cylinder>
     </link>
+    <gazebo reference="cylinder">
+        <material>Gazebo/Black</material>
+    </gazebo>
     <!-- ball castor-->
-    <joint name = "l_castor_joint" type = "fixed">
-        <parent link = "l_cylinder"/>
-        <child link = "l_castor"/>
+    <joint name = "castor_joint" type = "fixed">
+        <parent link = "cylinder"/>
+        <child link = "castor"/>
         <origin xyz = "0 0 -0.004" rpy = "0 0 0"/>
     </joint>
-    <link name = "l_castor">
+    <link name = "castor">
          <visual>
             <geometry>
@@ -128,3 +140,8 @@
         </xacro:inertial_sphere>
     </link>
+    <gazebo reference="castor">
+        <material>Gazebo/Orange</material>
+        <mu1 value="0.001"/>
+        <mu2 value="0.001"/>
+    </gazebo>
 </robot>
